File: hardware/LishuiFOC.sch (KiCad schematic (older format))
At the start: 105 parts

Commit message: add more things add and fix shunt
Signed-off-by: D3_M0N <chrisdietrich88@web.de>
Parts:
- added C? (x8): 100nF, symbol Device:C
- added C?: 15nF, symbol Device:C
- added D?: LED, symbol Device:LED
- added D?: 1N4148W, Diode_SMD:D_SOD-123, symbol Diode:1N4148W
- added J?: SPEED, symbol Connector_Generic:Conn_01x03
- added J?: Conn_01x02, symbol Connector_Generic:Conn_01x02
- added J?: PAS, symbol Connector_Generic:Conn_01x04
- added J?: THROTTLE, symbol Connector_Generic:Conn_01x03
- added J?: HALL, symbol Connector_Generic:Conn_01x05
- added R? (x3): 0.002, symbol Device:R_Shunt
- added R? (x7): 2.2k, symbol Device:R
- added R? (x3): 4.7k, symbol Device:R
- added R? (x3): 9.1k, symbol Device:R
- added R?: 5.1k 1%, symbol Device:R
- added R?: 75k 1%, symbol Device:R
- added R?: R, symbol Device:R
- R?: value R -> 100k
Connections:
- net labels added: SHUNT_UN, SHUNT_UW, SHUNT_VN, SHUNT_WN
- net labels removed: LED
- wire segments 231 -> 295
Other:
- note added: "22v-52v\n650uA"
- note added: "25v 10s leer\n42v full 10s \n30v 12s leer\n50,4v full 12s"
- note added: "3k3 10n??"
- note added: "5-3.3\n \n650uA"
- note added: "5v->3.3v\n \n360uA"
- note added: "PHASE CURRENT/HALL"
- note added: "RECALC"
- note added: "SENSORS"
- note removed: "PHASE CURRENT"
